Commit message: add moveit

File: so101_description/config/so101_position.ros2_control.xacro (robot description, xacro)
@@ -1,18 +1,25 @@
-<?xml version="1.0" ?>
+<?xml version="1.0"?>
 <robot xmlns:xacro="http://www.ros.org/wiki/xacro">
   <xacro:macro
-    name="ros2_control"
-    params="ros2_control_hardware_type usb_port prefix"
+    name="so101_ros2_control"
+    params="name prefix usb_port:=^|/dev/ttyUSB0 use_sim:=^|false use_fake_hardware:=^|false"
   >
-    <ros2_control name="so101" type="system">
-      <hardware>
-        <xacro:if value="${ros2_control_hardware_type == 'mock_components'}">
-          <plugin>mock_components/GenericSystem</plugin>
-        </xacro:if>
-        <xacro:if value="${ros2_control_hardware_type == 'real'}">
-          <plugin>feetech_ros2_driver/FeetechHardwareInterface</plugin>
-          <param name="usb_port">${usb_port}</param>
-        </xacro:if>
-      </hardware>
+    <ros2_control name="${name}" type="system">
+      <xacro:if value="$(arg use_sim)">
+        <hardware>
+          <plugin>gz_ros2_control/GazeboSimSystem</plugin>
+        </hardware>
+      </xacro:if>
+      <xacro:unless value="$(arg use_sim)">
+        <hardware>
+          <xacro:if value="${use_fake_hardware}">
+            <plugin>mock_components/GenericSystem</plugin>
+          </xacro:if>
+          <xacro:unless value="${use_fake_hardware}">
+            <plugin>feetech_ros2_driver/FeetechHardwareInterface</plugin>
+            <param name="usb_port">${usb_port}</param>
+          </xacro:unless>
+        </hardware>
+      </xacro:unless>
       <joint name="${prefix}shoulder_pan">
         <param name="initial_position">0.0</param>

File: so101_description/urdf/so101.urdf.xacro (robot description, xacro)
@@ -1,24 +1,27 @@
-<?xml version="1.0" ?>
+<?xml version="1.0"?>
 <robot xmlns:xacro="http://www.ros.org/wiki/xacro" name="so101">
-  <xacro:arg name="ros2_control_hardware_type" default="mock_components" />
-  <xacro:arg
-    name="ros2_control_file"
-    default="$(find so101_description)/urdf/so101.ros2_control.xacro"
-  />
-  <xacro:arg
-    name="urdf_file"
-    default="$(find so101_description)/urdf/so101_new_calib.urdf.xacro"
-  />
   <xacro:arg name="prefix" default="" />
-  <xacro:arg name="usb_port" default="/dev/LeRobotFollower" />
-  <!-- Robot description -->
-  <xacro:include filename="$(arg urdf_file)" />
-  <xacro:so101_new_calib prefix="$(arg prefix)" />
-  <!-- ros2_control description -->
-  <xacro:include filename="$(arg ros2_control_file)" />
-  <xacro:ros2_control
-    ros2_control_hardware_type="$(arg ros2_control_hardware_type)"
-    usb_port="$(arg usb_port)"
-    prefix="$(arg prefix)"
-  />
+  <xacro:arg name="use_sim" default="false" />
+  <xacro:arg name="use_fake_hardware" default="false" />
+  <xacro:arg name="usb_port" default="/dev/ttyUSB0" />
+  <xacro:arg name="ros2_control_type" default="so101_position" />
+  <xacro:include filename="$(find so101_description)/urdf/so101_new_calib.urdf.xacro" />
+  <xacro:include
+    filename="$(find so101_description)/config/$(arg ros2_control_type).ros2_control.xacro" />
+  <link name="world" />
+  <joint name="$(arg prefix)world_fixed" type="fixed">
+    <origin xyz="0 0 0" rpy="0 0 0" />
+    <parent link="world" />
+    <child link="$(arg prefix)base_link" />
+  </joint>
+  <xacro:so101 prefix="$(arg prefix)" />
+  <xacro:so101_ros2_control
+    name="so101_system" prefix="$(arg prefix)" use_sim="$(arg use_sim)"
+    use_fake_hardware="$(arg use_fake_hardware)"
+    usb_port="$(arg usb_port)" />
+  <gazebo>
+    <plugin filename="gz_ros2_control-system" name="gz_ros2_control::GazeboSimROS2ControlPlugin">
+      <parameters>$(find so101_description)/config/controller_manager.yaml</parameters>
+    </plugin>
+  </gazebo>
 </robot>

File: so101_description/urdf/so101_new_calib.urdf.xacro (robot description, xacro)
@@ -3,5 +3,5 @@
 <!-- Onshape https://cad.onshape.com/documents/7715cc284bb430fe6dab4ffd/w/4fd0791b683777b02f8d975a/e/826c553ede3b7592eb9ca800 -->
 <robot name="so101_new_calib" xmlns:xacro="http://www.ros.org/wiki/xacro">
-  <xacro:macro name="so101_new_calib" params="prefix">
+  <xacro:macro name="so101" params="prefix">
     <!-- Materials -->
     <material name="3d_printed">

Commit message: fix moveit config

File: so101_description/config/so101_position.ros2_control.xacro (robot description, xacro)
@@ -34,5 +34,5 @@
         <param name="id">2</param>
         <param name="p_cofficient">40</param>
-        <param name="offset">2100</param>
+        <param name="offset">2010</param>
         <param name="initial_position">0.0</param>
         <command_interface name="position" />
@@ -51,5 +51,5 @@
       <joint name="${prefix}wrist_flex">
         <param name="id">4</param>
-        <param name="offset">1946</param>
+        <param name="offset">2050</param>
         <param name="p_cofficient">4</param>
         <param name="initial_position">0.0</param>

File: so101_description/urdf/so101_new_calib.urdf.xacro (robot description, xacro)
@@ -381,5 +381,5 @@
       <child link="${prefix}lower_arm_link"/>
       <axis xyz="0 0 1"/>
-      <limit effort="10" velocity="10" lower="-1.69" upper="1.69"/>
+      <limit effort="10" velocity="10" lower="-1.69" upper="1.5966"/>
     </joint>
     <transmission name="${prefix}elbow_flex_trans">

Commit message: migrate teleop to a another repository

File: so101_description/config/so101_position.ros2_control.xacro (robot description, xacro)
@@ -3,6 +3,7 @@
   <xacro:macro
     name="so101_ros2_control"
-    params="name prefix usb_port:=^|/dev/ttyUSB0 use_sim:=^|false use_fake_hardware:=^|false"
+    params="name prefix usb_port:=^|/dev/ttyUSB0 use_sim:=^|false use_fake_hardware:=^|false initial_positions_file"
   >
+    <xacro:property name="initial_positions" value="${xacro.load_yaml(initial_positions_file)['initial_positions']}"/>
     <ros2_control name="${name}" type="system">
       <xacro:if value="$(arg use_sim)">
@@ -23,6 +24,6 @@
       </xacro:unless>
       <joint name="${prefix}shoulder_pan">
-        <param name="initial_position">0.0</param>
         <param name="id">1</param>
+        <param name="initial_position">${initial_positions['shoulder_pan']}</param>
         <param name="p_cofficient">10</param>
         <param name="offset">2048</param>
@@ -33,7 +34,7 @@
       <joint name="${prefix}shoulder_lift">
         <param name="id">2</param>
+        <param name="initial_position">${initial_positions['shoulder_lift']}</param>
         <param name="p_cofficient">16</param>
         <param name="offset">1990</param>
-        <param name="initial_position">0.0</param>
         <command_interface name="position" />
         <state_interface name="position" />
@@ -42,7 +43,7 @@
       <joint name="${prefix}elbow_flex">
         <param name="id">3</param>
+        <param name="initial_position">${initial_positions['elbow_flex']}</param>
         <param name="offset">2068</param>
         <param name="p_cofficient">20</param>
-        <param name="initial_position">0.0</param>
         <command_interface name="position" />
         <state_interface name="position" />
@@ -51,7 +52,7 @@
       <joint name="${prefix}wrist_flex">
         <param name="id">4</param>
+        <param name="initial_position">${initial_positions['wrist_flex']}</param>
         <param name="offset">2048</param>
         <param name="p_cofficient">20</param>
-        <param name="initial_position">0.0</param>
         <command_interface name="position" />
         <state_interface name="position" />
@@ -60,7 +61,7 @@
       <joint name="${prefix}wrist_roll">
         <param name="id">5</param>
+        <param name="initial_position">${initial_positions['wrist_roll']}</param>
         <param name="offset">1982</param>
         <param name="p_cofficient">16</param>
-        <param name="initial_position">0.0</param>
         <command_interface name="position" />
         <state_interface name="position" />
@@ -69,7 +70,7 @@
       <joint name="${prefix}gripper">
         <param name="id">6</param>
+        <param name="initial_position">${initial_positions['gripper']}</param>
         <param name="offset">2048</param>
         <param name="p_cofficient">16</param>
-        <param name="initial_position">0.0</param>
         <command_interface name="position" />
         <state_interface name="position" />

File: so101_description/urdf/so101.urdf.xacro (robot description, xacro)
@@ -6,4 +6,5 @@
   <xacro:arg name="usb_port" default="/dev/ttyUSB0" />
   <xacro:arg name="ros2_control_type" default="so101_position" />
+  <xacro:arg name="initial_positions_file" default="initial_positions.yaml" />
   <xacro:include filename="$(find so101_description)/urdf/so101_new_calib.urdf.xacro" />
   <xacro:include
@@ -19,5 +20,6 @@
     name="so101_system" prefix="$(arg prefix)" use_sim="$(arg use_sim)"
     use_fake_hardware="$(arg use_fake_hardware)"
-    usb_port="$(arg usb_port)" />
+    usb_port="$(arg usb_port)"
+    initial_positions_file="$(arg initial_positions_file)" />
   <gazebo>
     <plugin filename="gz_ros2_control-system" name="gz_ros2_control::GazeboSimROS2ControlPlugin">
